Commit message: feat(launch): add launch-files for world, robot, teleop, mapping, rviz

File: urdf/lw_mse6_bot.xacro (robot description, xacro)
@@ -2,6 +2,6 @@
 <robot name="lw_mse6_bot"
     xmlns:xacro="http://www.ros.org/wiki/xacro">
-    <xacro:include filename="$(find udacity_bot)/urdf/lw_mse6_bot.gazebo"/>
-    <xacro:include filename="$(find udacity_bot)/urdf/macros.xacro" />
+    <xacro:include filename="$(find slam_project)/urdf/lw_mse6_bot.gazebo"/>
+    <xacro:include filename="$(find slam_project)/urdf/macros.xacro" />
     <xacro:property name="PI" value="3.1415926535897931"/>
     <xacro:property name="epsilon" value="0.0001"/>
@@ -50,4 +50,9 @@
         <child link="camera"/>
     </joint>
+    <joint name="camera_rgbd_joint" type="fixed">
+        <origin xyz="0 0 0" rpy="-${pi/2} 0 -${pi/2}"/>
+        <parent link="camera"/>
+        <child link="camera_rgbd_frame"/>
+    </joint>
     <joint name="hokuyo_joint" type="fixed">
         <origin xyz="0.2 0.0 0.15" rpy="0.0 0.0 0.0"/>
@@ -65,5 +70,5 @@
             <origin xyz="0.0 0.0 0.0" rpy="0.0 0.0 0.0"/>
             <geometry>
-                <mesh filename="package://udacity_bot/meshes/lw_mse6_chassis.dae"/>
+                <mesh filename="package://slam_project/meshes/lw_mse6_chassis.dae"/>
             </geometry>
         </visual>
@@ -76,5 +81,5 @@
             <origin xyz="0.0 0.0 0.0" rpy="0.0 0.0 0.0"/>
             <geometry>
-                <mesh filename="package://udacity_bot/meshes/lw_mse6_chassis.dae"/>
+                <mesh filename="package://slam_project/meshes/lw_mse6_chassis.dae"/>
             </geometry>
         </collision>
@@ -172,4 +177,5 @@
         </collision>
     </link>
+    <link name="camera_rgbd_frame"></link>
     <link name="hokuyo">
         <inertial>
@@ -181,5 +187,5 @@
             <origin xyz="0.0 0.0 0.0" rpy="0.0 0.0 0.0"/>
             <geometry>
-                <mesh filename="package://udacity_bot/meshes/hokuyo.dae"/>
+                <mesh filename="package://slam_project/meshes/hokuyo.dae"/>
             </geometry>
         </visual>
